File: hardware/pcb/kicad/safeboat-termica-v1.kicad_sch (KiCad schematic)
At the start: 32 parts, among them J1 USB (JST-PH 4), J2 +12V (borne KF350), Q1 SI2301, SW1 BOOT, SW2 RST, U1 ESP32-C3-MINI-1-N4, U2 AP63203WU-7, U3 MLX90640ESF-BAA

Commit message: PCB térmica rev. 2: 40×40 mm, 4 camadas, 8–32 V (MP4560), antena com recortes, 4 furos, pads de alimentação
Pedidos da reunião de 22/10: nada metálico ao lado da antena; diretrizes Espressif
(recortes laterais na antena, keep-out em 4 camadas, plano GND sob o módulo);
trilhas a 90° (snap_angle no DSN); planos internos sólidos In1 GND / In2 3V3
(roteador vê só F/B); isolamento 0,2 mm; furos M2,5 longe da antena; PPTC mantido;
MP4560 + SMBJ33A + 4,7 µF/100 V para 8–32 V; borne removido (pads P1/P2).
DRC 0/0/0, ERC 0, netlist esquemático × PCB 0 diferenças. BOM com todos os códigos.
Pacote de revisão regenerado (inclui planos internos).

Co-Authored-By: Claude Fable 5.1 <noreply@anthropic.com>
Parts:
- removed J2: +12V (borne KF350), SAFEBOAT:KF350-3.5-2P, symbol Connector_Generic:Conn_01x02
- removed U2: AP63203WU-7, Package_TO_SOT_SMD:TSOT-23-6, symbol SAFEBOAT:AP63203
- added C11: 4.7u/100V, Capacitor_SMD:C_1210_3225Metric, symbol Device:C
- added C12: 1n, Capacitor_SMD:C_0603_1608Metric, symbol Device:C
- added D4: SS36, Diode_SMD:D_SMA, symbol Device:D_Schottky
- added P1: +VIN 8-32V (pad), SAFEBOAT:WirePad_P1, symbol SAFEBOAT:WirePad
- added P2: GND (pad), SAFEBOAT:WirePad_P2, symbol SAFEBOAT:WirePad
- added R10: 15k, Resistor_SMD:R_0603_1608Metric, symbol Device:R
- added R11: 200k, Resistor_SMD:R_0603_1608Metric, symbol Device:R
- added R12: 68k, Resistor_SMD:R_0603_1608Metric, symbol Device:R
- added R9: 47k, Resistor_SMD:R_0603_1608Metric, symbol Device:R
- added U2: MP4560DN-LF-Z, Package_SO:HSOP-8-1EP_3.9x4.9mm_P1.27mm_EP2.41x3.1mm_ThermalVias, symbol SAFEBOAT:MP4560
- C5: value 10u/50V -> 4.7u/100V
- D1: value SMAJ26A -> SMBJ33A; footprint Diode_SMD:D_SMA -> Diode_SMD:D_SMB
- L1: value 4.7u SWPA4020S -> 10u SWPA5040S; footprint Inductor_SMD:L_Sunlord_SWPA4020S -> Inductor_SMD:L_Sunlord_SWPA5040S
- R7: value 200k -> 330k
- R8: value 20k -> 15k
Connections:
- net 3V3: now also R9.1
- net BST: now also U2.8 (BST)
- net GND: now also C11.2, C12.2, D4.2 (A), P2.1, R10.2, R11.2, U2.5 (GND), U2.9 (EP)
- net SW: now also D4.1 (K), U2.1 (SW)
- net VIN: now also C11.1, U2.7 (VIN)
- net VIN_RAW: now also P1.1
- new net COMP: R12.1, U2.3 (COMP)
- new net COMP_C: C12.1, R12.2
- new net FB: R10.1, R9.2, U2.4 (FB)
- new net FREQ: R11.1, U2.6 (FREQ)
- no-connect marks 22 -> 23
Other:
- note added: "1 · ALIMENTACAO — +8-32 V (pads P1/P2, fio soldado) -> F1 PPTC 0,5 A -> D1 TVS SMBJ33A -> D2 SS34 (inversao) -> VIN -> U2 MP4560 (500 kHz, EN flutuante = liga) -> L1 10 uH / D4 SS36 -> 3V3 (FB 47k/15k) · USB J1 -> D3 SS14 -> VIN · R7/R8 leem VIN/23 no ADC (GPIO0)"
- note added: "Redes por label (mesma netlist pino a pino de make_board.py). Placa 40 x 40 mm, 4 camadas (In1 GND, In2 3V3); sensor no lado B (frente), resto no lado F (re). Montagem completa JLCPCB (2 lados)."
- note added: "SAFEBOAT TERMICA v2 — camera termica MLX90640 110 + ESP32-C3, 8-32 V do barco, 4 camadas · esquematico p/ revisao"
- note removed: "1 · ALIMENTACAO — +12 V (borne J2) -> F1 PPTC 0,5 A -> D1 TVS SMBJ26A -> D2 SS34 (inversao) -> VIN -> U2 AP63203 (EN=VIN, FB=VOUT) -> L1 4,7 uH -> 3V3 · USB J1 -> D3 SS14 -> VIN (bancada) · R7/R8 leem VIN no ADC (GPIO0)"
- note removed: "Redes por label (mesma netlist pino a pino de make_board.py). Placa quadrada 32 x 32 mm; sensor no lado B (frente), resto no lado F (re). Montagem completa JLCPCB (2 lados)."
- note removed: "SAFEBOAT TERMICA v1 — camera termica MLX90640 + ESP32-C3, 12 V do barco · esquematico p/ revisao"
- title: SAFEBOAT TERMICA v1 — camera termica MLX90640 + ESP32-C3 -> SAFEBOAT TERMICA v2 — camera termica MLX90640 110 + ESP32-C3, 8-32 V
